Commit message: fix: separate Kyon lower-leg and foot collision proxies
Crop the primitive lower-leg boxes so the spherical foot proxies remain the dedicated ground-contact geometry.

File: robots/kyon_description/urdf/kyon_quadruped.urdf (robot description, URDF)
Before this commit: robot kyon, 25 links, 24 joints
Links:
- link knee_pitch_1_link: geometry collision box size=0.079951 0.2741 0.043661; visual mesh filename=package://example-robot-data/robots/kyon_description/meshes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 scale=-0.001 0.001 0.001
- link knee_pitch_2_link: geometry collision box size=0.079951 0.2741 0.043661; visual mesh filename=package://example-robot-data/robots/kyon_description/meshes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 scale=0.001 0.001 0.001
- link knee_pitch_3_link: geometry collision box size=0.079951 0.2741 0.043661; visual mesh filename=package://example-robot-data/robots/kyon_description/meshes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 scale=-0.001 0.001 0.001
- link knee_pitch_4_link: geometry collision box size=0.079951 0.2741 0.043661; visual mesh filename=package://example-robot-data/robots/kyon_description/meshes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 scale=0.001 0.001 0.001

File: robots/kyon_description/urdf/kyon_quadruped_manipulator.urdf (robot description, URDF)
Before this commit: robot kyon, 39 links, 38 joints
Links:
- link knee_pitch_1_link: geometry collision box size=0.079951 0.2741 0.043661; visual mesh filename=package://example-robot-data/robots/kyon_description/meshes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 scale=-0.001 0.001 0.001
- link knee_pitch_2_link: geometry collision box size=0.079951 0.2741 0.043661; visual mesh filename=package://example-robot-data/robots/kyon_description/meshes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 scale=0.001 0.001 0.001
- link knee_pitch_3_link: geometry collision box size=0.079951 0.2741 0.043661; visual mesh filename=package://example-robot-data/robots/kyon_description/meshes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 scale=-0.001 0.001 0.001
- link knee_pitch_4_link: geometry collision box size=0.079951 0.2741 0.043661; visual mesh filename=package://example-robot-data/robots/kyon_description/meshes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 scale=0.001 0.001 0.001
